Commit message: separeted chassis and robotHead
Co-authored-by: Copilot <copilot@github.com>

File: src/vision_voyager_description/urdf/vision_voyager.urdf.xacro (robot description, xacro)
@@ -21,5 +21,5 @@
       <origin xyz="0 0 0" rpy="0 0 0"/>
       <geometry>
-        <mesh filename="package://vision_voyager_description/3d_mesh_models/3D_vv_chassis.obj" scale="1 1 1"/>
+        <mesh filename="package://vision_voyager_description/3d_mesh_models/chassis.obj" scale="1 1 1"/>
       </geometry>
     </visual>
@@ -51,6 +51,7 @@
   <link name="tilt_link">
     <visual>
-      <geometry><box size="0.02 0.03 0.02"/></geometry>
-      <material name="blue"/>
+      <geometry>
+        <mesh filename="package://vision_voyager_description/3d_mesh_models/head_tilt.obj" scale="1 1 1"/>
+      </geometry>
     </visual>
     <inertial>

Commit message: added camera module
Co-authored-by: Copilot <copilot@github.com>

File: src/vision_voyager_description/urdf/vision_voyager.urdf.xacro (robot description, xacro)
@@ -66,4 +66,22 @@
     <axis xyz="0 1 0"/>
     <limit lower="-0.78" upper="0.78" effort="1.0" velocity="1.0"/>
+  </joint>
+  <link name="camera_link">
+    <visual>
+      <geometry><box size="0.02 0.02 0.02"/></geometry>
+      <material name="black"/>
+    </visual>
+    <collision>
+      <geometry><box size="0.02 0.02 0.02"/></geometry>
+    </collision>
+    <inertial>
+      <mass value="0.01"/>
+      <inertia ixx="1e-5" ixy="0" ixz="0" iyy="1e-5" iyz="0" izz="1e-5"/>
+    </inertial>
+  </link>
+  <joint name="camera_joint" type="fixed">
+    <parent link="tilt_link"/>
+    <child link="camera_link"/>
+    <origin xyz="0.05 0 0.02" rpy="0 0 0"/>
   </joint>
   <link name="ultrasonic_link">
@@ -216,4 +234,23 @@
     </sensor>
   </gazebo>
+  <gazebo reference="camera_link">
+    <sensor name="camera" type="camera">
+      <pose>0 0 0 0 0 0</pose>
+      <gz_frame_id>camera_link</gz_frame_id>
+      <topic>/camera/image_raw</topic>
+      <always_on>true</always_on>
+      <update_rate>30</update_rate>
+      <visualize>true</visualize>
+      <camera>
+        <horizontal_fov>1.047</horizontal_fov>
+        <image>
+          <width>640</width>
+          <height>480</height>
+          <format>R8G8B8</format>
+        </image>
+        <clip><near>0.01</near><far>100</far></clip>
+      </camera>
+    </sensor>
+  </gazebo>
   <xacro:macro name="line_follower_gz" params="prefix">
     <gazebo reference="line_follower_${prefix}">
