Commit message: fresh new start with ROS 2 Jazzy and Gazebo Harmonic

File: src/vision_voyager_description/urdf/vision_voyager.urdf.xacro (robot description, xacro)
@@ -1,86 +1,122 @@
 <?xml version="1.0"?>
 <robot name="vision_voyager" xmlns:xacro="http://www.ros.org/wiki/xacro">
-  <xacro:property name="chassis_l" value="0.17"/>
-  <xacro:property name="chassis_w" value="0.10"/>
-  <xacro:property name="chassis_h" value="0.04"/>
-  <xacro:property name="wheel_r" value="0.033"/>
-  <xacro:property name="wheel_w" value="0.025"/>
-  <material name="blue"> <color rgba="0 0 0.8 1"/> </material>
-  <material name="black"> <color rgba="0 0 0 1"/> </material>
+  <xacro:property name="chassis_mass" value="0.8"/>
+  <xacro:property name="wheel_mass" value="0.1"/>
+  <xacro:property name="wheel_radius" value="0.032"/>
+  <xacro:property name="wheel_width" value="0.015"/>
+  <xacro:property name="wheelbase" value="0.12"/>
+  <xacro:property name="track_width" value="0.1"/>
+  <material name="blue"><color rgba="0.1 0.4 0.8 1"/></material>
+  <material name="black"><color rgba="0.05 0.05 0.05 1"/></material>
   <link name="base_footprint"/>
   <joint name="base_joint" type="fixed">
     <parent link="base_footprint"/>
-    <child link="base_link"/>
-    <origin xyz="0 0 ${wheel_r}" rpy="0 0 0"/>
+    <child link="chassis"/>
+    <origin xyz="0 0 ${wheel_radius}" rpy="0 0 0"/>
   </joint>
-  <link name="base_link">
+  <link name="chassis">
     <visual>
-      <origin xyz="0 0 0.02" rpy="0 0 0"/>
-      <geometry> <box size="${chassis_l} ${chassis_w} ${chassis_h}"/> </geometry>
+      <geometry><box size="0.16 0.09 0.01"/></geometry>
       <material name="blue"/>
     </visual>
     <collision>
-      <origin xyz="0 0 0.02" rpy="0 0 0"/>
-      <geometry> <box size="${chassis_l} ${chassis_w} ${chassis_h}"/> </geometry>
+      <geometry><box size="0.16 0.09 0.01"/></geometry>
     </collision>
     <inertial>
-      <origin xyz="0 0 0.02" rpy="0 0 0"/>
-      <mass value="0.5"/>
-      <inertia ixx="0.001" ixy="0" ixz="0" iyy="0.001" iyz="0" izz="0.001"/>
+      <mass value="${chassis_mass}"/>
+      <inertia ixx="0.00054" ixy="0" ixz="0" iyy="0.00171" iyz="0" izz="0.00224"/>
     </inertial>
   </link>
-  <xacro:macro name="wheel" params="prefix x y">
-    <link name="${prefix}_wheel">
+  <xacro:macro name="rear_wheel" params="prefix y_reflect">
+    <link name="rear_${prefix}_wheel">
       <visual>
         <origin rpy="${pi/2} 0 0" xyz="0 0 0"/>
-        <geometry> <cylinder radius="${wheel_r}" length="${wheel_w}"/> </geometry>
+        <geometry><cylinder radius="${wheel_radius}" length="${wheel_width}"/></geometry>
         <material name="black"/>
       </visual>
       <collision>
         <origin rpy="${pi/2} 0 0" xyz="0 0 0"/>
-        <geometry> <cylinder radius="${wheel_r}" length="${wheel_w}"/> </geometry>
+        <geometry><cylinder radius="${wheel_radius}" length="${wheel_width}"/></geometry>
       </collision>
       <inertial>
-        <mass value="0.1"/>
-        <inertia ixx="1e-4" ixy="0" ixz="0" iyy="1e-4" iyz="0" izz="1e-4"/>
+        <mass value="${wheel_mass}"/>
+        <inertia ixx="0.00003" ixy="0" ixz="0" iyy="0.00003" iyz="0" izz="0.00005"/>
       </inertial>
     </link>
-    <joint name="${prefix}_wheel_joint" type="continuous">
-      <parent link="base_link"/>
-      <child link="${prefix}_wheel"/>
-      <origin xyz="${x} ${y} 0" rpy="0 0 0"/>
+    <joint name="rear_${prefix}_wheel_joint" type="continuous">
+      <parent link="chassis"/>
+      <child link="rear_${prefix}_wheel"/>
+      <origin xyz="-${wheelbase/2} ${y_reflect * track_width/2} 0" rpy="0 0 0"/>
       <axis xyz="0 1 0"/>
     </joint>
+    <gazebo reference="rear_${prefix}_wheel">
+      <mu1>1.0</mu1>
+      <mu2>1.0</mu2>
+      <material>Gazebo/Black</material>
+    </gazebo>
   </xacro:macro>
-  <xacro:wheel prefix="front_left"  x="0.06"  y="0.06"/>
-  <xacro:wheel prefix="front_right" x="0.06"  y="-0.06"/>
-  <xacro:wheel prefix="rear_left"   x="-0.06" y="0.06"/>
-  <xacro:wheel prefix="rear_right"  x="-0.06" y="-0.06"/>
+  <xacro:macro name="front_wheel" params="prefix y_reflect">
+    <link name="front_${prefix}_steer_link">
+      <inertial><mass value="0.01"/><inertia ixx="0.000001" ixy="0" ixz="0" iyy="0.000001" iyz="0" izz="0.000001"/></inertial>
+    </link>
+    <joint name="front_${prefix}_steer_joint" type="revolute">
+      <parent link="chassis"/>
+      <child link="front_${prefix}_steer_link"/>
+      <origin xyz="${wheelbase/2} ${y_reflect * track_width/2} 0" rpy="0 0 0"/>
+      <axis xyz="0 0 1"/>
+      <limit lower="-0.52" upper="0.52" effort="5.0" velocity="1.0"/>
+    </joint>
+    <link name="front_${prefix}_wheel">
+      <visual>
+        <origin rpy="${pi/2} 0 0" xyz="0 0 0"/>
+        <geometry><cylinder radius="${wheel_radius}" length="${wheel_width}"/></geometry>
+        <material name="black"/>
+      </visual>
+      <collision>
+        <origin rpy="${pi/2} 0 0" xyz="0 0 0"/>
+        <geometry><cylinder radius="${wheel_radius}" length="${wheel_width}"/></geometry>
+      </collision>
+      <inertial>
+        <mass value="${wheel_mass}"/>
+        <inertia ixx="0.00003" ixy="0" ixz="0" iyy="0.00003" iyz="0" izz="0.00005"/>
+      </inertial>
+    </link>
+    <joint name="front_${prefix}_wheel_joint" type="continuous">
+      <parent link="front_${prefix}_steer_link"/>
+      <child link="front_${prefix}_wheel"/>
+      <axis xyz="0 1 0"/>
+    </joint>
+    <gazebo reference="front_${prefix}_wheel">
+      <mu1>1.0</mu1>
+      <mu2>1.0</mu2>
+      <material>Gazebo/Black</material>
+    </gazebo>
+  </xacro:macro>
+  <xacro:rear_wheel prefix="left" y_reflect="1"/>
+  <xacro:rear_wheel prefix="right" y_reflect="-1"/>
+  <xacro:front_wheel prefix="left" y_reflect="1"/>
+  <xacro:front_wheel prefix="right" y_reflect="-1"/>
   <gazebo>
-    <plugin name="skid_steer_drive" filename="libgazebo_ros_diff_drive.so">
-      <ros>
-        <remapping>cmd_vel:=cmd_vel</remapping>
-        <remapping>odom:=odom</remapping>
-      </ros>
-      <update_rate>30</update_rate>
-      <num_wheel_pairs>2</num_wheel_pairs>
-      <left_joint>front_left_wheel_joint</left_joint>
+    <plugin
+      filename="gz-sim-ackermann-steering-system"
+      name="gz::sim::systems::AckermannSteering">
       <left_joint>rear_left_wheel_joint</left_joint>
-      <right_joint>front_right_wheel_joint</right_joint>
       <right_joint>rear_right_wheel_joint</right_joint>
-      <wheel_separation>0.12</wheel_separation>
-      <wheel_diameter>0.066</wheel_diameter>
-      <max_wheel_torque>20</max_wheel_torque>
-      <max_wheel_acceleration>1.0</max_wheel_acceleration>
-      <publish_odom>true</publish_odom>
-      <publish_odom_tf>true</publish_odom_tf>
-      <odometry_frame>odom</odometry_frame>
-      <robot_base_frame>base_footprint</robot_base_frame>
+      <left_steering_joint>front_left_steer_joint</left_steering_joint>
+      <right_steering_joint>front_right_steer_joint</right_steering_joint>
+      <wheel_separation>${track_width}</wheel_separation>
+      <wheel_radius>${wheel_radius}</wheel_radius>
+      <topic>cmd_vel</topic>
+      <min_velocity>-1.0</min_velocity>
+      <max_velocity>1.0</max_velocity>
+      <min_acceleration>-3.0</min_acceleration>
+      <max_acceleration>3.0</max_acceleration>
     </plugin>
   </gazebo>
-  <gazebo reference="base_link"><material>Gazebo/Blue</material></gazebo>
-  <gazebo reference="front_left_wheel"><material>Gazebo/Black</material></gazebo>
-  <gazebo reference="front_right_wheel"><material>Gazebo/Black</material></gazebo>
-  <gazebo reference="rear_left_wheel"><material>Gazebo/Black</material></gazebo>
-  <gazebo reference="rear_right_wheel"><material>Gazebo/Black</material></gazebo>
+  <gazebo>
+    <plugin
+      filename="gz-sim-joint-state-publisher-system"
+      name="gz::sim::systems::JointStatePublisher">
+    </plugin>
+  </gazebo>
 </robot>

Commit message: added ultrasonic sensor

File: src/vision_voyager_description/urdf/vision_voyager.urdf.xacro (robot description, xacro)
@@ -9,4 +9,5 @@
   <material name="blue"><color rgba="0.1 0.4 0.8 1"/></material>
   <material name="black"><color rgba="0.05 0.05 0.05 1"/></material>
+  <material name="grey"><color rgba="0.5 0.5 0.5 1"/></material>
   <link name="base_footprint"/>
   <joint name="base_joint" type="fixed">
@@ -28,4 +29,22 @@
     </inertial>
   </link>
+  <link name="ultrasonic_link">
+    <visual>
+      <geometry><box size="0.02 0.05 0.02"/></geometry>
+      <material name="grey"/>
+    </visual>
+    <collision>
+      <geometry><box size="0.02 0.05 0.02"/></geometry>
+    </collision>
+    <inertial>
+      <mass value="0.01"/>
+      <inertia ixx="1e-5" ixy="0" ixz="0" iyy="1e-5" iyz="0" izz="1e-5"/>
+    </inertial>
+  </link>
+  <joint name="ultrasonic_joint" type="fixed">
+    <parent link="chassis"/>
+    <child link="ultrasonic_link"/>
+    <origin xyz="0.08 0 0.03" rpy="0 0 0"/>
+  </joint>
   <xacro:macro name="rear_wheel" params="prefix y_reflect">
     <link name="rear_${prefix}_wheel">
@@ -50,13 +69,8 @@
       <axis xyz="0 1 0"/>
     </joint>
-    <gazebo reference="rear_${prefix}_wheel">
-      <mu1>1.0</mu1>
-      <mu2>1.0</mu2>
-      <material>Gazebo/Black</material>
-    </gazebo>
   </xacro:macro>
   <xacro:macro name="front_wheel" params="prefix y_reflect">
     <link name="front_${prefix}_steer_link">
-      <inertial><mass value="0.01"/><inertia ixx="0.000001" ixy="0" ixz="0" iyy="0.000001" iyz="0" izz="0.000001"/></inertial>
+      <inertial><mass value="0.01"/><inertia ixx="1e-6" ixy="0" ixz="0" iyy="1e-6" iyz="0" izz="1e-6"/></inertial>
     </link>
     <joint name="front_${prefix}_steer_joint" type="revolute">
@@ -87,9 +101,4 @@
       <axis xyz="0 1 0"/>
     </joint>
-    <gazebo reference="front_${prefix}_wheel">
-      <mu1>1.0</mu1>
-      <mu2>1.0</mu2>
-      <material>Gazebo/Black</material>
-    </gazebo>
   </xacro:macro>
   <xacro:rear_wheel prefix="left" y_reflect="1"/>
@@ -98,7 +107,5 @@
   <xacro:front_wheel prefix="right" y_reflect="-1"/>
   <gazebo>
-    <plugin
-      filename="gz-sim-ackermann-steering-system"
-      name="gz::sim::systems::AckermannSteering">
+    <plugin filename="gz-sim-ackermann-steering-system" name="gz::sim::systems::AckermannSteering">
       <left_joint>rear_left_wheel_joint</left_joint>
       <right_joint>rear_right_wheel_joint</right_joint>
@@ -108,15 +115,33 @@
       <wheel_radius>${wheel_radius}</wheel_radius>
       <topic>cmd_vel</topic>
-      <min_velocity>-1.0</min_velocity>
-      <max_velocity>1.0</max_velocity>
-      <min_acceleration>-3.0</min_acceleration>
-      <max_acceleration>3.0</max_acceleration>
+    </plugin>
+    <plugin filename="gz-sim-joint-state-publisher-system" name="gz::sim::systems::JointStatePublisher"/>
+    <plugin filename="gz-sim-sensors-system" name="gz::sim::systems::Sensors">
+      <render_engine>ogre2</render_engine>
     </plugin>
   </gazebo>
-  <gazebo>
-    <plugin
-      filename="gz-sim-joint-state-publisher-system"
-      name="gz::sim::systems::JointStatePublisher">
-    </plugin>
+  <gazebo reference="ultrasonic_link">
+    <sensor name="hc_sr04" type="gpu_lidar">
+      <gz_frame_id>ultrasonic_link</gz_frame_id>
+      <topic>/ultrasonic/scan</topic>
+      <always_on>true</always_on>
+      <update_rate>10</update_rate>
+      <visualize>true</visualize>
+      <ray>
+        <scan>
+          <horizontal>
+            <samples>3</samples>
+            <resolution>1</resolution>
+            <min_angle>-0.15</min_angle>
+            <max_angle>0.15</max_angle>
+          </horizontal>
+        </scan>
+        <range>
+          <min>0.05</min>
+          <max>3.0</max>
+          <resolution>0.01</resolution>
+        </range>
+      </ray>
+    </sensor>
   </gazebo>
 </robot>

Commit message: added line follower

File: src/vision_voyager_description/urdf/vision_voyager.urdf.xacro (robot description, xacro)
@@ -10,4 +10,5 @@
   <material name="black"><color rgba="0.05 0.05 0.05 1"/></material>
   <material name="grey"><color rgba="0.5 0.5 0.5 1"/></material>
+  <material name="red"><color rgba="0.8 0.1 0.1 1"/></material>
   <link name="base_footprint"/>
   <joint name="base_joint" type="fixed">
@@ -47,4 +48,24 @@
     <origin xyz="0.08 0 0.03" rpy="0 0 0"/>
   </joint>
+  <xacro:macro name="line_follower_link" params="prefix y_off">
+    <link name="line_follower_${prefix}">
+      <visual>
+        <geometry><box size="0.01 0.01 0.005"/></geometry>
+        <material name="red"/>
+      </visual>
+      <inertial>
+        <mass value="0.001"/>
+        <inertia ixx="1e-7" ixy="0" ixz="0" iyy="1e-7" iyz="0" izz="1e-7"/>
+      </inertial>
+    </link>
+    <joint name="line_follower_${prefix}_joint" type="fixed">
+      <parent link="chassis"/>
+      <child link="line_follower_${prefix}"/>
+      <origin xyz="0.075 ${y_off} -0.005" rpy="0 ${pi/2} 0"/>
+    </joint>
+  </xacro:macro>
+  <xacro:line_follower_link prefix="left"   y_off="0.02"/>
+  <xacro:line_follower_link prefix="center" y_off="0.0"/>
+  <xacro:line_follower_link prefix="right"  y_off="-0.02"/>
   <xacro:macro name="rear_wheel" params="prefix y_reflect">
     <link name="rear_${prefix}_wheel">
@@ -116,5 +137,5 @@
       <topic>cmd_vel</topic>
     </plugin>
-    <plugin filename="gz-sim-joint-state-publisher-system" name="gz::sim::systems::JointStatePublisher"/>
+      <plugin filename="gz-sim-joint-state-publisher-system" name="gz::sim::systems::JointStatePublisher"/>
     <plugin filename="gz-sim-sensors-system" name="gz::sim::systems::Sensors">
       <render_engine>ogre2</render_engine>
@@ -145,3 +166,26 @@
     </sensor>
   </gazebo>
+  <xacro:macro name="line_follower_gz" params="prefix">
+    <gazebo reference="line_follower_${prefix}">
+      <sensor name="line_follower_${prefix}" type="camera">
+        <gz_frame_id>line_follower_${prefix}</gz_frame_id>
+        <always_on>true</always_on>
+        <update_rate>30</update_rate>
+        <visualize>true</visualize>
+        <topic>/line_follower/${prefix}</topic>
+        <camera>
+          <horizontal_fov>0.1</horizontal_fov>
+          <image>
+            <width>1</width>
+            <height>1</height>
+            <format>R8G8B8</format>
+          </image>
+          <clip><near>0.001</near><far>0.10</far></clip>
+        </camera>
+      </sensor>
+    </gazebo>
+  </xacro:macro>
+  <xacro:line_follower_gz prefix="left"/>
+  <xacro:line_follower_gz prefix="center"/>
+  <xacro:line_follower_gz prefix="right"/>
 </robot>

Commit message: added pan/tilt movement for camera

File: src/vision_voyager_description/urdf/vision_voyager.urdf.xacro (robot description, xacro)
@@ -30,4 +30,38 @@
     </inertial>
   </link>
+  <link name="pan_link">
+    <visual>
+      <geometry><box size="0.03 0.03 0.03"/></geometry>
+      <material name="grey"/>
+    </visual>
+    <inertial>
+      <mass value="0.05"/>
+      <inertia ixx="1e-5" ixy="0" ixz="0" iyy="1e-5" iyz="0" izz="1e-5"/>
+    </inertial>
+  </link>
+  <joint name="pan_joint" type="revolute">
+    <parent link="chassis"/>
+    <child link="pan_link"/>
+    <origin xyz="0.04 0 0.02" rpy="0 0 0"/>
+    <axis xyz="0 0 1"/>
+    <limit lower="-1.57" upper="1.57" effort="1.0" velocity="1.0"/>
+  </joint>
+  <link name="tilt_link">
+    <visual>
+      <geometry><box size="0.02 0.03 0.02"/></geometry>
+      <material name="blue"/>
+    </visual>
+    <inertial>
+      <mass value="0.05"/>
+      <inertia ixx="1e-5" ixy="0" ixz="0" iyy="1e-5" iyz="0" izz="1e-5"/>
+    </inertial>
+  </link>
+  <joint name="tilt_joint" type="revolute">
+    <parent link="pan_link"/>
+    <child link="tilt_link"/>
+    <origin xyz="0.01 0 0.025" rpy="0 0 0"/>
+    <axis xyz="0 1 0"/>
+    <limit lower="-0.78" upper="0.78" effort="1.0" velocity="1.0"/>
+  </joint>
   <link name="ultrasonic_link">
     <visual>
@@ -137,7 +171,15 @@
       <topic>cmd_vel</topic>
     </plugin>
-      <plugin filename="gz-sim-joint-state-publisher-system" name="gz::sim::systems::JointStatePublisher"/>
+    <plugin filename="gz-sim-joint-state-publisher-system" name="gz::sim::systems::JointStatePublisher"/>
     <plugin filename="gz-sim-sensors-system" name="gz::sim::systems::Sensors">
       <render_engine>ogre2</render_engine>
+    </plugin>
+    <plugin filename="gz-sim-joint-position-controller-system" name="gz::sim::systems::JointPositionController">
+      <joint_name>pan_joint</joint_name>
+      <topic>/model/vision_voyager/joint/pan_joint/cmd_pos</topic>
+    </plugin>
+    <plugin filename="gz-sim-joint-position-controller-system" name="gz::sim::systems::JointPositionController">
+      <joint_name>tilt_joint</joint_name>
+      <topic>/model/vision_voyager/joint/tilt_joint/cmd_pos</topic>
     </plugin>
   </gazebo>

Commit message: chassis + wheel integration

File: src/vision_voyager_description/urdf/vision_voyager.urdf.xacro (robot description, xacro)
@@ -19,6 +19,8 @@
   <link name="chassis">
     <visual>
-      <geometry><box size="0.16 0.09 0.01"/></geometry>
-      <material name="blue"/>
+      <origin xyz="0 0 0" rpy="0 0 0"/>
+      <geometry>
+        <mesh filename="package://vision_voyager_description/3d_mesh_models/3D_vv_chassis.obj" scale="1 1 1"/>
+      </geometry>
     </visual>
     <collision>
@@ -102,9 +104,14 @@
   <xacro:line_follower_link prefix="center" y_off="0.0"/>
   <xacro:line_follower_link prefix="right"  y_off="-0.02"/>
+  <xacro:macro name="wheel_geometry">
+    <geometry>
+      <mesh filename="package://vision_voyager_description/3d_mesh_models/vv_wheel.obj" scale="1 1 1"/>
+    </geometry>
+  </xacro:macro>
   <xacro:macro name="rear_wheel" params="prefix y_reflect">
     <link name="rear_${prefix}_wheel">
       <visual>
-        <origin rpy="${pi/2} 0 0" xyz="0 0 0"/>
-        <geometry><cylinder radius="${wheel_radius}" length="${wheel_width}"/></geometry>
+        <origin rpy="0 ${pi/2} ${(1 - y_reflect) * pi / 2}" xyz="0 0 0"/>
+        <xacro:wheel_geometry/>
         <material name="black"/>
       </visual>
@@ -138,6 +145,6 @@
     <link name="front_${prefix}_wheel">
       <visual>
-        <origin rpy="${pi/2} 0 0" xyz="0 0 0"/>
-        <geometry><cylinder radius="${wheel_radius}" length="${wheel_width}"/></geometry>
+        <origin rpy="0 ${pi/2} ${(1 - y_reflect) * pi / 2}" xyz="0 0 0"/>
+        <xacro:wheel_geometry/>
         <material name="black"/>
       </visual>
@@ -231,3 +238,36 @@
   <xacro:line_follower_gz prefix="center"/>
   <xacro:line_follower_gz prefix="right"/>
+  <xacro:macro name="wheel_gazebo_material" params="prefix side">
+    <gazebo reference="${prefix}_${side}_wheel">
+      <visual>
+        <material>
+          <pbr>
+            <metal>
+              <albedo_map>package://vision_voyager_description/3d_mesh_models/vv_wheel.png</albedo_map>
+              <roughness>0.6</roughness>
+              <metalness>0.1</metalness>
+            </metal>
+          </pbr>
+        </material>
+      </visual>
+    </gazebo>
+  </xacro:macro>
+  <xacro:wheel_gazebo_material prefix="front" side="left"/>
+  <xacro:wheel_gazebo_material prefix="front" side="right"/>
+  <xacro:wheel_gazebo_material prefix="rear" side="left"/>
+  <xacro:wheel_gazebo_material prefix="rear" side="right"/>
+  <gazebo reference="chassis">
+      <visual>
+          <material>
+              <ambient>1 1 1 1</ambient>
+              <diffuse>1 1 1 1</diffuse>
+              <specular>0.5 0.5 0.5 1</specular>
+              <pbr>
+                  <metal>
+                      <albedo_map>package://vision_voyager_description/3d_mesh_models/chassis_Texture.png</albedo_map>
+                  </metal>
+              </pbr>
+          </material>
+      </visual>
+  </gazebo>
 </robot>

Commit message: improved wheel rotation velocity

File: src/vision_voyager_description/urdf/vision_voyager.urdf.xacro (robot description, xacro)
@@ -160,5 +160,5 @@
       <origin xyz="${wheelbase/2} ${y_reflect * track_width/2} 0" rpy="0 0 0"/>
       <axis xyz="0 0 1"/>
-      <limit lower="-0.52" upper="0.52" effort="5.0" velocity="1.0"/>
+      <limit lower="-0.52" upper="0.52" effort="10.0" velocity="20.0"/>
     </joint>
     <link name="front_${prefix}_wheel">
